File: 4k-mania-keypad.kicad_pcb (KiCad board)
At the start: 2 copper layers, 112 x 47.2 mm, 43 parts, among them J1 USB_C_Receptacle_USB2.0, J2 Pico Ezmate, J3 Pico Ezmate, J4 Pico Ezmate, J5 Pico Ezmate, SW1 EC11E18244A5, SW2 EC11E18244A5, SW3 MX_SW_HS, SW4 MX_SW_HS, SW5 MX_SW_HS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

Commit message: main pcb routing finished
Parts:
- SW3, SW4, SW5, SW6: moved to B.Cu
- moved C7 118.5 mm to (183.5, 86.0)
- moved C8 115.6 mm to (180.5, 93.0), turned to -90 degrees
- moved C11 114.5 mm to (178.7, 81.5), turned to 90 degrees
- moved C6 110.6 mm to (171.9, 83.5), turned to 180 degrees
- moved C9 110.4 mm to (175.0, 81.5), turned to 90 degrees
- moved C10 109.1 mm to (174.1, 91.5), turned to 180 degrees
- moved C12 105.9 mm to (170.4, 86.4), turned to 180 degrees
- moved C13 97.6 mm to (183.5, 85.0)
- moved C14 86.3 mm to (171.9, 84.5), turned to 180 degrees
- moved C15 84.6 mm to (170.4, 87.4), turned to 180 degrees
- moved C3 84.4 mm to (160.0, 87.0), turned to -90 degrees
- moved U4 79.3 mm to (163.4, 87.1), turned to 90 degrees
- moved J2 69.4 mm to (146.7, 94.6)
- moved U1 62.6 mm to (177.7, 86.7), turned to 90 degrees
- moved C4 62.5 mm to (184.4, 88.3), turned to 90 degrees
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Connections:
- D2 pad 1: /rsw0(0) -> /rsw1(1)
- R3 pad 1: GND -> Net-(C5-Pad2)
- SW1 pad A: /rotA(1) -> /rotA(0)
- SW1 pad B: /rotB(1) -> /rotB(0)
- SW1 pad S2: /rsw1(1) -> /rsw0(0)
- SW2 pad A: /rotA(0) -> /rotA(1)
- SW2 pad B: /rotB(0) -> /rotB(1)
- U1 pad 11: /rotB(1) -> /rotB(0)
- U1 pad 12: /rotA(1) -> /rotA(0)
- U1 pad 15: /rsw1(1) -> /rotB(1)
- U1 pad 16: /rsw0(1) -> /rotA(1)
- U1 pad 2: /col0(0) -> /col0(1)
- U1 pad 3: /col1(0) -> /col1(1)
- U1 pad 4: /row0(0) -> /row0(1)
- U1 pad 5: /col0(1) -> /row0(0)
- U1 pad 6: /col1(1) -> /col1(0)
- U1 pad 7: /row0(1) -> /col0(0)
- U1 pad 8: /rotB(0) -> /rsw1(1)
- U1 pad 9: /rotA(0) -> /rsw0(1)
- U2 pad 3: /USB_D+ -> /USB_D-
- U2 pad 4: /USB_D- -> /USB_D+
Routing:
- net /rsw0(0): track 0.00 -> 98.1 mm, vias 0 -> 2
- net /rsw1(0): track 0.00 -> 88.8 mm, vias 0 -> 2
- net /rotB(0): track 0.00 -> 81.7 mm, vias 0 -> 2
- net /rotA(0): track 0.00 -> 79.4 mm, vias 0 -> 2
- net +3.3V: track 0.00 -> 68.5 mm, vias 0 -> 2
- net /reset: track 0.00 -> 41.2 mm, vias 0 -> 2
- net /rsw0(1): track 0.00 -> 39.5 mm
- net /USB_D+: track 0.00 -> 37.6 mm
- net /USB_D-: track 0.00 -> 37.4 mm
- net /col0(0): track 0.00 -> 37.0 mm
- net /col1(0): track 0.00 -> 34.9 mm
- net /row0(0): track 0.00 -> 32.8 mm
- net /rsw1(1): track 0.00 -> 30.6 mm
- net /row0(1): track 0.00 -> 22.9 mm
- net /col1(1): track 0.00 -> 20.8 mm
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- added copper zone on B.Cu, net GND
- added copper zone on F.Cu, net GND
Other:
- board size 112 x 47.2 mm -> 112 x 48.5 mm

Commit message: First finished draft
Parts:
- D3, D4, D5, D6, J4, J5: moved to B.Cu
- moved D5 19.0 mm to (170.7, 111.5), turned to 90 degrees
- moved D6 17.2 mm to (189.6, 114.9), turned to 90 degrees
- moved D3 14.3 mm to (97.0, 114.5), turned to 90 degrees
- moved D4 11.5 mm to (116.2, 114.6), turned to 90 degrees
- moved J5 9.12 mm to (171.5, 116.0), turned to 90 degrees
- moved J4 8.45 mm to (130.1, 115.7), turned to -90 degrees
- moved J3 1.80 mm to (156.2, 94.6)
- moved J2 0.45 mm to (146.2, 94.6)
- moved C8 0.37 mm to (180.5, 93.4)
Connections:
- J5 pad 3: Net-(D5-A) -> Net-(J5-Pin_3)
- SW5 pad 2: Net-(D5-A) -> Net-(J5-Pin_3)
Routing:
- net Net-(J5-Pin_2): track 0.00 -> 39.8 mm
- net Net-(D3-K): track 0.00 -> 31.8 mm
- net Net-(D5-K): track 0.00 -> 23.3 mm
- net Net-(J4-Pin_2): track 0.00 -> 23.0 mm
- net Net-(J5-Pin_3): track 0.00 -> 15.6 mm
- net Net-(J4-Pin_1): track 0.00 -> 9.24 mm
- net Net-(D6-A): track 0.00 -> 5.49 mm
- net +3.3V: track 68.5 -> 73.7 mm, vias 2 -> 3
- net Net-(D3-A): track 0.00 -> 5.15 mm
- net Net-(D4-A): track 0.00 -> 5.11 mm
- net Net-(D5-A): track 0.00 -> 2.09 mm
- net /col1(1): track 20.8 -> 22.6 mm
- net /row0(1): track 22.9 -> 24.7 mm
- net /col0(1): track 18.5 -> 20.3 mm
- net +1V1: track 19.2 -> 18.7 mm

Commit message: fixed many issues and generated fab files
Parts:
- added R5: 27.4, Resistor_SMD:R_0402_1005Metric, F.Cu at (168.0, 82.0)
- added R6: 27.4, Resistor_SMD:R_0402_1005Metric, F.Cu at (169.0, 82.0)
- added REF**: mousebites 1mm, marbastlib-various:mousebites_1mm, F.Cu at (114.2, 97.5)
- added REF**: mousebites 1mm, marbastlib-various:mousebites_1mm, F.Cu at (186.5, 97.5)
- C1: value 13uF -> 1uF
- C10, C11, C13, C14, C6, C7, C8, C9: value 0.1uF -> 100nF
- C12, C15: value 2.2uF -> 1uF
- C2: value 14uF -> 1uF
- C4, C5: value 22pF -> 27pF
- D1, D2, D3, D4, D5, D6: value D_Small -> d
- R4: value 10k -> 1k; footprint Resistor_SMD:R_0805_2012Metric -> Resistor_SMD:R_0402_1005Metric
- SW7: footprint Connector_PinSocket_2.54mm:PinSocket_1x02_P2.54mm_Vertical -> random-keyboard-parts:SKQG-1155865
- moved SW7 4.17 mm to (141.0, 87.6), turned to 0 degrees
- moved D5 3.64 mm to (169.7, 108.0)
- moved D6 3.64 mm to (188.6, 111.4)
- moved J5 3.64 mm to (170.5, 112.5)
- moved SW5 3.64 mm to (177.1, 108.0)
- moved SW6 3.64 mm to (196.0, 108.0)
- moved D3 3.42 mm to (97.1, 111.1)
- moved D4 3.42 mm to (116.3, 111.1)
- moved J4 3.42 mm to (130.2, 112.2)
- moved SW3 3.42 mm to (104.7, 108.1)
- moved SW4 3.42 mm to (123.7, 108.1)
- moved D2 0.71 mm to (204.5, 95.5)
- moved R4 0.66 mm to (147.7, 89.1)
- moved SW2 0.50 mm to (190.5, 84.5)
- moved SW1 0.25 mm to (111.5, 89.5)
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Connections:
- U1 pad 46: /USB_D- -> Net-(U1-D-)
- U1 pad 47: /USB_D+ -> Net-(U1-D+)
Routing:
- net /USB_D+: track 37.6 -> 28.8 mm
- net Net-(U1-D+): track 0.00 -> 8.35 mm
- net /USB_D-: track 37.4 -> 29.7 mm
- net Net-(U1-D-): track 0.00 -> 7.53 mm
- net Net-(J4-Pin_2): track 23.0 -> 23.9 mm
- net Net-(D1-A): track 12.0 -> 11.1 mm
- net /rsw1(1): track 30.6 -> 29.9 mm
- net Net-(D5-K): track 23.3 -> 24.0 mm
- net /reset: track 41.2 -> 41.8 mm
- net /rotB(1): track 10.3 -> 9.74 mm
- net +3.3V: track 73.7 -> 73.2 mm
- net Net-(D2-A): track 5.51 -> 6.01 mm
Other:
- board size 112 x 48.5 mm -> 112 x 45 mm
