File: 4k-mania-keypad.kicad_sch (KiCad schematic)
At the start: 43 parts, among them J1 USB_C_Receptacle_USB2.0, J5 Pico Ezmate, J6 Pico Ezmate, SW1 EC11E18244A5, SW2 EC11E18244A5, SW3 MX_SW_HS, SW3 SW_Push, SW4 MX_SW_HS, SW5 MX_SW_HS, SW6 MX_SW_HS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

Commit message: main pcb routing finished
Connections:
- net GND: no longer R3.1
- net USB_D+: now also U2.4 (IO3); no longer U2.3 (IO2)
- net USB_D-: now also U2.3 (IO2); no longer U2.4 (IO3)
- net col0(0): now also U1.7 (GPIO5); no longer U1.2 (GPIO0)
- net col0(1): now also U1.2 (GPIO0); no longer U1.5 (GPIO3)
- net col1(0): now also U1.6 (GPIO4); no longer U1.3 (GPIO1)
- net col1(1): now also U1.3 (GPIO1); no longer U1.6 (GPIO4)
- net rotA(0): now also SW2.A, U1.12 (GPIO9); no longer SW1.A, U1.9 (GPIO7)
- net rotA(1): now also SW1.A, U1.16 (GPIO13); no longer SW2.A, U1.12 (GPIO9)
- net rotB(0): now also SW2.B, U1.11 (GPIO8); no longer SW1.B, U1.8 (GPIO6)
- net rotB(1): now also SW1.B, U1.15 (GPIO12); no longer SW2.B, U1.11 (GPIO8)
- net row0(0): now also U1.5 (GPIO3); no longer U1.4 (GPIO2)
- net row0(1): now also U1.4 (GPIO2); no longer U1.7 (GPIO5)
- net rsw0(0): now also SW2.S2; no longer D2.1 (K)
- net rsw0(1): now also U1.9 (GPIO7); no longer U1.16 (GPIO13)
- net rsw1(1): now also D2.1 (K), U1.8 (GPIO6); no longer SW2.S2, U1.15 (GPIO12)
- net at C3.2, Y1.1: now also R3.1
Other:
- moved on the sheet: R3

Commit message: First finished draft
Connections:
- net at D5.2 (A), SW5.1: no longer J5.3 (Pin_3), SW5.2
- new net: J5.3 (Pin_3), SW5.2

Commit message: fixed many issues and generated fab files
Parts:
- removed C11, C13, C14, C6, C7, C8, C9: 0.1uF, Capacitor_SMD:C_0402_1005Metric, symbol Device:C_Small
- removed C12, C15: 2.2uF, Capacitor_SMD:C_0402_1005Metric, symbol Device:C_Small
- added C5 (x7): 100nF, Capacitor_SMD:C_0402_1005Metric, symbol Device:C_Small
- added C5 (x2): 1uF, Capacitor_SMD:C_0402_1005Metric, symbol Device:C_Small
- added R5, R6: 27.4, Resistor_SMD:R_0402_1005Metric, symbol Device:R_Small
- C1: value 13uF -> 1uF; Vendor (none) -> C52923
- C2: value 14uF -> 1uF; Vendor (none) -> C52923
- C2, C3: value 22pF -> 27pF; LCSC C1555 -> (none); Vendor (none) -> C1557
- C3: Vendor (none) -> C307331
- C5: value 0.1uF -> 100nF; Vendor (none) -> C307331
- D1, D2, D3, D4, D5, D6: value D_Small -> d; Vendor (none) -> C191023
- F1: Vendor (none) -> C355568
- J1: Vendor (none) -> C223907
- R1, R2: Vendor (none) -> C103086
- R3: Vendor (none) -> C11702
- R4: value 10k -> 1k; footprint Resistor_SMD:R_0805_2012Metric -> Resistor_SMD:R_0402_1005Metric; Vendor (none) -> C11702
- SW1, SW2: Vendor (none) -> C255515
- SW3: footprint Connector_PinSocket_2.54mm:PinSocket_1x02_P2.54mm_Vertical -> random-keyboard-parts:SKQG-1155865; Vendor (none) -> C388858
- U1: Vendor (none) -> C2040
- U2: Vendor (none) -> C85364
- U3: Vendor (none) -> C5446
- U4: Vendor (none) -> C97521
- Y1: Vendor (none) -> C9002
Connections:
- net +1V1: now also C5.1, C5.1, C5.1
- net +3.3V: now also C5.1, C5.1, C5.1, C5.1, C5.1, C5.1
- net GND: now also C5.2, C5.2, C5.2, C5.2, C5.2, C5.2, C5.2, C5.2, C5.2
- net USB_D+: now also R5.1; no longer U1.47 (D+)
- net USB_D-: now also R6.1; no longer U1.46 (D-)
- new net: R6.2, U1.46 (D-)
- new net: R5.2, U1.47 (D+)
